File: cncshitter/cncshitter.kicad_pcb (KiCad board)
At the start: 2 copper layers, 51 parts, among them J1 24V_IN, J2 5V_IN, J3 DB25_Male_MountingHoles, J4 SPINDLE_PWM_ENC, J5 SPINDLE_ENABLE, J6 EMERGENCY_PROBE_ENABLE, J7 AXIS_XYZ, K1 SANYOU_SRD_Form_C, K2 SANYOU_SRD_Form_C, U1 EMERGENCY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

Commit message: v2
Parts:
- added H1: MountingHole, MountingHole:MountingHole_3mm_Pad, F.Cu at (28.0, 86.0)
- added H2: MountingHole, MountingHole:MountingHole_3mm_Pad, F.Cu at (26.0, 36.0)
- added H3: MountingHole, MountingHole:MountingHole_3mm_Pad, F.Cu at (132.0, 86.0)
- added H4: MountingHole, MountingHole:MountingHole_3mm_Pad, F.Cu at (134.0, 36.0)
- J1, J2, J3, J4, J5, J6, J7: moved to B.Cu
- moved J4 101.5 mm to (53.8, 29.0), turned to 0 degrees
- moved J5 96.6 mm to (80.5, 29.0), turned to 0 degrees
- moved J6 90.7 mm to (31.8, 29.2), turned to 0 degrees
- moved R7 75.6 mm to (69.2, 38.3), turned to 90 degrees
- moved C1 74.5 mm to (64.9, 37.2), turned to 180 degrees
- moved R3 74.2 mm to (125.0, 74.3), turned to 90 degrees
- moved J2 70.8 mm to (118.1, 91.4), turned to 180 degrees
- moved K2 70.7 mm to (90.7, 41.7), turned to 180 degrees
- moved C2 69.1 mm to (64.9, 41.0), turned to 180 degrees
- moved U3 68.2 mm to (126.2, 65.2), turned to 90 degrees
- moved R11 67.3 mm to (51.6, 55.7), turned to 270 degrees
- moved R8 66.5 mm to (69.2, 43.6), turned to 90 degrees
- moved R14 66.0 mm to (117.3, 74.3), turned to 90 degrees
- moved D2 63.8 mm to (94.5, 45.5), turned to 90 degrees
- moved C3 63.7 mm to (64.9, 44.8), turned to 180 degrees
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Connections:
- J4 pad 1: Net-(J4-Pad1) -> GND
- J4 pad 2: Net-(C1-Pad1) -> Net-(J4-Pad2)
- J4 pad 4: Net-(J4-Pad4) -> Net-(C1-Pad1)
- J4 pad 5: GND -> Net-(J4-Pad5)
- R7 pad 2: Net-(J4-Pad1) -> Net-(J4-Pad5)
- U4 pad 2: Net-(U4-Pad2) -> /LPT_GND
- U5 pad 2: Net-(J4-Pad4) -> Net-(J4-Pad2)
Routing:
- net Net-(D2-Pad2): track 27.6 -> 141.8 mm, vias 0 -> 2
- net Net-(J4-Pad4): track 86.8 -> 0.00 mm
- net VCC: track 189.3 -> 116.3 mm
- net Net-(J4-Pad2): track 0.00 -> 37.6 mm
- net /ENABLE: track 6.14 -> 41.4 mm
- net Net-(R6-Pad2): track 35.7 -> 2.86 mm
- net /SPINDLE_ENC: track 56.5 -> 24.8 mm, vias 2 -> 0
- net Net-(R25-Pad2): track 34.5 -> 2.86 mm
- net Net-(J7-Pad1): track 14.9 -> 46.2 mm, vias 0 -> 2
- net /AXIS_X_DIR: track 5.33 -> 36.5 mm
- net Net-(R24-Pad2): track 32.7 -> 2.86 mm
- net GND: track 192.0 -> 162.5 mm, vias 2 -> 0
- net Net-(J6-Pad1): track 59.2 -> 30.9 mm
- net Net-(R3-Pad2): track 31.2 -> 2.86 mm
- net /PROBE: track 58.5 -> 30.5 mm, vias 2 -> 0
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Other:
- board outline added: 116 x 74 mm
- net class Default: via_dia 0.8 -> 1.2; via_drill 0.4 -> 1
- net class pwr: via_dia 0.8 -> 1.2; via_drill 0.4 -> 1

Commit message: v2 fixes
Routing:
- net Net-(R10-Pad2): track 0.00 -> 2.79 mm
Changed lines of the file:
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@@
     (thickness 1.6)
     (drawings 6)
-    (tracks 306)
+    (tracks 307)
     (zones 0)
     (modules 55)
@@
   (segment (start 66.548 60.386) (end 66.548 53.34) (width 0.3) (layer F.Cu) (net 46))
   (segment (start 34.29 60.066) (end 34.29 57.277) (width 0.3) (layer F.Cu) (net 47))
+  (segment (start 42.418 60.071) (end 42.418 57.277) (width 0.3) (layer F.Cu) (net 48))
   (segment (start 51.562 60.066) (end 51.562 57.204) (width 0.3) (layer F.Cu) (net 49))
   (segment (start 117.348 72.771) (end 117.348 69.916) (width 0.3) (layer F.Cu) (net 50))

Commit message: v2 fixes 2
Parts:
- moved J6 0.80 mm to (32.5, 29.0)
Routing:
- net Net-(J6-Pad4): track 21.6 -> 16.3 mm
- net /LPT_GND: track 204.0 -> 206.0 mm
- net Net-(J6-Pad2): track 38.2 -> 40.1 mm
- net Net-(J6-Pad1): track 30.9 -> 32.3 mm
- net Net-(J6-Pad3): track 7.31 -> 7.88 mm
Changed lines of the file:
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@@
     (thickness 1.6)
     (drawings 6)
-    (tracks 307)
+    (tracks 312)
     (zones 0)
     (modules 55)
@@
   )
   (module Connector_Phoenix_MC_HighVoltage:PhoenixContact_MC_1,5_4-G-5.08_1x04_P5.08mm_Horizontal (layer B.Cu)
-    (at 31.75 29.21)
+    (at 32.512 28.956)
     (descr "Generic Phoenix Contact connector footprint for: MC_1,5/4-G-5.08; number of pins: 04; pin pitch: 5.08mm; Angled || order number: 1836202 8A 320V")
     (tags "phoenix_contact connector MC_01x04_G_5.08mm")
@@
   (segment (start 31.75 77.75) (end 31.75 69.596) (width 1) (layer F.Cu) (net 9))
   (segment (start 40 86) (end 31.75 77.75) (width 1) (layer F.Cu) (net 9))
-  (segment (start 31.75 68.985998) (end 32.917998 67.818) (width 1) (layer F.Cu) (net 9))
-  (segment (start 31.75 69.596) (end 31.75 68.985998) (width 1) (layer F.Cu) (net 9))
   (segment (start 127.508 67.916) (end 127.508 69.916) (width 1) (layer F.Cu) (net 9))
   (segment (start 127.41 67.818) (end 127.508 67.916) (width 1) (layer F.Cu) (net 9))
@@
   (segment (start 77.724 67.818) (end 86.868 67.818) (width 1) (layer F.Cu) (net 9))
   (segment (start 86.868 67.818) (end 96.012 67.818) (width 1) (layer F.Cu) (net 9))
-  (segment (start 49.022 69.596) (end 49.022 68.072) (width 1) (layer F.Cu) (net 9))
-  (segment (start 49.022 68.072) (end 49.276 67.818) (width 1) (layer F.Cu) (net 9))
-  (segment (start 49.276 67.818) (end 60.198 67.818) (width 1) (layer F.Cu) (net 9))
-  (segment (start 39.878 69.601) (end 39.878 68.072) (width 1) (layer F.Cu) (net 9))
-  (segment (start 39.878 68.072) (end 39.624 67.818) (width 1) (layer F.Cu) (net 9))
-  (segment (start 32.917998 67.818) (end 39.624 67.818) (width 1) (layer F.Cu) (net 9))
-  (segment (start 39.624 67.818) (end 49.276 67.818) (width 1) (layer F.Cu) (net 9))
+  (segment (start 31.75 67.596) (end 32.036 67.31) (width 1) (layer F.Cu) (net 9))
+  (segment (start 31.75 69.596) (end 31.75 67.596) (width 1) (layer F.Cu) (net 9))
+  (segment (start 59.69 67.31) (end 60.198 67.818) (width 1) (layer F.Cu) (net 9))
+  (segment (start 49.022 69.596) (end 49.022 67.596) (width 1) (layer F.Cu) (net 9))
+  (segment (start 49.022 67.596) (end 49.022 67.31) (width 1) (layer F.Cu) (net 9))
+  (segment (start 49.022 67.31) (end 59.69 67.31) (width 1) (layer F.Cu) (net 9))
+  (segment (start 39.878 67.601) (end 39.878 67.31) (width 1) (layer F.Cu) (net 9))
+  (segment (start 39.878 69.601) (end 39.878 67.601) (width 1) (layer F.Cu) (net 9))
+  (segment (start 32.036 67.31) (end 39.878 67.31) (width 1) (layer F.Cu) (net 9))
+  (segment (start 39.878 67.31) (end 49.022 67.31) (width 1) (layer F.Cu) (net 9))
   (segment (start 51.943 75.365) (end 51.943 77.089) (width 1) (layer F.Cu) (net 10))
   (segment (start 34.29 75.111) (end 42.418 75.111) (width 1) (layer F.Cu) (net 10))
@@
   (segment (start 76.528 32.946) (end 80.518 28.956) (width 0.3) (layer F.Cu) (net 30))
   (segment (start 76.528 35.606) (end 76.528 32.946) (width 0.3) (layer F.Cu) (net 30))
-  (segment (start 53.848 41.656) (end 46.736 41.656) (width 0.3) (layer F.Cu) (net 31))
-  (segment (start 46.736 41.656) (end 44.45 39.37) (width 0.3) (layer F.Cu) (net 31))
-  (segment (start 46.99 30.11) (end 44.45 32.65) (width 0.3) (layer F.Cu) (net 31))
-  (segment (start 44.45 32.65) (end 44.45 39.37) (width 0.3) (layer F.Cu) (net 31))
-  (segment (start 46.99 29.21) (end 46.99 30.11) (width 0.3) (layer F.Cu) (net 31))
-  (segment (start 41.91 33.394) (end 41.91 29.21) (width 0.3) (layer F.Cu) (net 32))
-  (segment (start 39.698 35.606) (end 41.91 33.394) (width 0.3) (layer F.Cu) (net 32))
-  (segment (start 39.878 58.771) (end 36.987 55.88) (width 0.3) (layer F.Cu) (net 33))
-  (segment (start 39.878 60.071) (end 39.878 58.771) (width 0.3) (layer F.Cu) (net 33))
-  (segment (start 36.987 55.88) (end 33.02 55.88) (width 0.3) (layer F.Cu) (net 33))
-  (segment (start 33.02 55.88) (end 32.25001 55.11001) (width 0.3) (layer F.Cu) (net 33))
-  (segment (start 36.83 31.31) (end 36.83 29.21) (width 0.3) (layer F.Cu) (net 33))
-  (segment (start 32.25001 35.88999) (end 36.83 31.31) (width 0.3) (layer F.Cu) (net 33))
-  (segment (start 32.25001 55.11001) (end 32.25001 35.88999) (width 0.3) (layer F.Cu) (net 33))
-  (segment (start 31.75 29.21) (end 31.75 60.066) (width 0.3) (layer F.Cu) (net 34))
+  (segment (start 48.006 37.592) (end 52.07 41.656) (width 0.3) (layer F.Cu) (net 31))
+  (segment (start 48.006 31.31) (end 48.006 37.592) (width 0.3) (layer F.Cu) (net 31))
+  (segment (start 52.07 41.656) (end 53.848 41.656) (width 0.3) (layer F.Cu) (net 31))
+  (segment (start 47.752 28.956) (end 47.752 31.056) (width 0.3) (layer F.Cu) (net 31))
+  (segment (start 47.752 31.056) (end 48.006 31.31) (width 0.3) (layer F.Cu) (net 31))
+  (segment (start 42.672 32.632) (end 39.698 35.606) (width 0.3) (layer F.Cu) (net 32))
+  (segment (start 42.672 28.956) (end 42.672 32.632) (width 0.3) (layer F.Cu) (net 32))
+  (segment (start 37.592 31.75) (end 37.592 28.956) (width 0.3) (layer F.Cu) (net 33))
+  (segment (start 32.004 37.338) (end 37.592 31.75) (width 0.3) (layer F.Cu) (net 33))
+  (segment (start 38.688 60.071) (end 36.83 58.213) (width 0.3) (layer F.Cu) (net 33))
+  (segment (start 36.83 58.213) (end 36.83 55.88) (width 0.3) (layer F.Cu) (net 33))
+  (segment (start 39.878 60.071) (end 38.688 60.071) (width 0.3) (layer F.Cu) (net 33))
+  (segment (start 36.83 55.88) (end 32.258 55.88) (width 0.3) (layer F.Cu) (net 33))
+  (segment (start 32.004 55.626) (end 32.004 37.338) (width 0.3) (layer F.Cu) (net 33))
+  (segment (start 32.258 55.88) (end 32.004 55.626) (width 0.3) (layer F.Cu) (net 33))
+  (segment (start 32.512 28.956) (end 30.734 30.734) (width 0.3) (layer F.Cu) (net 34))
+  (segment (start 31.75 58.766) (end 31.75 60.066) (width 0.3) (layer F.Cu) (net 34))
+  (segment (start 30.734 57.75) (end 31.75 58.766) (width 0.3) (layer F.Cu) (net 34))
+  (segment (start 30.734 30.734) (end 30.734 57.75) (width 0.3) (layer F.Cu) (net 34))
   (segment (start 117.348 28.956) (end 117.348 54.556) (width 0.3) (layer F.Cu) (net 35))
   (segment (start 112.268 52.2335) (end 109.728 54.7735) (width 0.3) (layer F.Cu) (net 36))

Commit message: v2 drc pass
Parts:
- moved J6 0.13 mm to (32.4, 29.0)
Routing:
- net Net-(J3-Pad0): track 0.00 -> 50.9 mm
Changed lines of the file:
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@@
     (thickness 1.6)
     (drawings 6)
-    (tracks 312)
+    (tracks 316)
     (zones 0)
     (modules 55)
@@
   )
   (module Connector_Phoenix_MC_HighVoltage:PhoenixContact_MC_1,5_4-G-5.08_1x04_P5.08mm_Horizontal (layer B.Cu)
-    (at 32.512 28.956)
+    (at 32.385 28.956)
     (descr "Generic Phoenix Contact connector footprint for: MC_1,5/4-G-5.08; number of pins: 04; pin pitch: 5.08mm; Angled || order number: 1836202 8A 320V")
     (tags "phoenix_contact connector MC_01x04_G_5.08mm")
@@
   (segment (start 113.03 90.54) (end 119.75 83.82) (width 1) (layer F.Cu) (net 10))
   (segment (start 113.03 91.44) (end 113.03 90.54) (width 1) (layer F.Cu) (net 10))
+  (segment (start 48.725 90.02) (end 53.193 94.488) (width 0.3) (layer F.Cu) (net 11))
+  (segment (start 53.193 94.488) (end 91.44 94.488) (width 0.3) (layer F.Cu) (net 11))
+  (segment (start 91.44 94.405) (end 95.825 90.02) (width 0.3) (layer F.Cu) (net 11))
+  (segment (start 91.44 94.488) (end 91.44 94.405) (width 0.3) (layer F.Cu) (net 11))
   (segment (start 34.29 72.136) (end 35.814 73.66) (width 0.3) (layer F.Cu) (net 16))
   (segment (start 35.814 73.66) (end 45.72 73.66) (width 0.3) (layer F.Cu) (net 16))

Commit message: v3 smaller
Parts:
- removed H2: MountingHole, MountingHole:MountingHole_3mm_Pad
- removed J3: DB25_Male_MountingHoles, Connector_Dsub:DSUB-25_Male_Horizontal_P2.77x2.84mm_EdgePinOffset7.70mm_Housed_MountingHolesOffset9.12mm
- moved J1 20.6 mm to (123.2, 49.5), turned to 270 degrees
- moved H4 7.01 mm to (127.0, 35.6)
- moved H1 6.36 mm to (34.3, 85.1)
- moved H3 5.08 mm to (127.0, 85.1)
- moved J2 3.59 mm to (117.1, 88.0)
Routing:
- net Net-(J3-Pad0): track 50.9 -> 0.00 mm
- net Net-(D2-Pad2): track 141.8 -> 105.3 mm
- net GND: track 162.5 -> 137.7 mm
- net VCC: track 116.3 -> 92.7 mm
- net /LPT_VCC: track 112.3 -> 104.6 mm
- net /PROBE: track 30.5 -> 23.3 mm
- net /LPT_GND: track 206.0 -> 212.3 mm
- net Net-(J7-Pad2): track 39.5 -> 34.4 mm
- net /EMERGENCY: track 33.7 -> 28.7 mm
- net /SPINDLE_PWM: track 14.1 -> 9.15 mm
- net /AXIS_Z_STEP: track 14.2 -> 9.23 mm
- net /SPINDLE_ENABLE: track 16.6 -> 12.4 mm
- net /AXIS_Z_DIR: track 16.7 -> 12.6 mm
- net Net-(D1-Pad2): track 106.3 -> 102.2 mm
- net Net-(J6-Pad4): track 16.3 -> 20.1 mm
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Other:
- board size 116 x 74 mm -> 104 x 70 mm
- net class Default: trace_width 0.3 -> 0.4

Commit message: v3 fixed
Parts:
- added J3: DB25_Male_MountingHoles, Connector_Dsub:DSUB-25_Male_Horizontal_P2.77x2.84mm_EdgePinOffset7.70mm_Housed_MountingHolesOffset9.12mm, B.Cu at (88.9, 83.8)
Changed lines of the file:
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@@
     (tracks 339)
     (zones 0)
-    (modules 53)
-    (nets 58)
+    (modules 54)
+    (nets 64)
   )
   (page A4)
@@
   (net 56 "Net-(J4-Pad2)")
   (net 57 "Net-(J4-Pad5)")
+  (net 58 "Net-(J3-Pad0)")
+  (net 59 "Net-(J3-Pad17)")
+  (net 60 "Net-(J3-Pad16)")
+  (net 61 "Net-(J3-Pad15)")
+  (net 62 "Net-(J3-Pad14)")
+  (net 63 "Net-(J3-Pad11)")
   (net_class Default "This is the default net class."
     (clearance 0.2)
@@
     (add_net "Net-(D2-Pad1)")
     (add_net "Net-(D2-Pad2)")
+    (add_net "Net-(J3-Pad0)")
+    (add_net "Net-(J3-Pad11)")
+    (add_net "Net-(J3-Pad14)")
+    (add_net "Net-(J3-Pad15)")
+    (add_net "Net-(J3-Pad16)")
+    (add_net "Net-(J3-Pad17)")
     (add_net "Net-(J4-Pad2)")
     (add_net "Net-(J4-Pad5)")
@@
     (add_net VCC)
   )
+  (module Connector_Dsub:DSUB-25_Male_Horizontal_P2.77x2.84mm_EdgePinOffset7.70mm_Housed_MountingHolesOffset9.12mm (layer B.Cu)
+    (at 88.9 83.82 180)
+    (descr "25-pin D-Sub connector, horizontal/angled (90 deg), THT-mount, male, pitch 2.77x2.84mm, pin-PCB-offset 7.699999999999999mm, distance of mounting holes 47.1mm, distance of mounting holes to PCB edge 9.12mm, see https://disti-assets.s3.amazonaws.com/tonar/files/datasheets/16730.pdf")
+    (tags "25-pin D-Sub connector horizontal angled 90deg THT male pitch 2.77x2.84mm pin-PCB-offset 7.699999999999999mm mounting-holes-distance 47.1mm mounting-hole-offset 47.1mm")
+    (fp_text reference J3 (at 16.62 2.8 180) (layer B.SilkS)
+      (effects (font (size 1 1) (thickness 0.15)) (justify mirror))
+    )
+    (fp_text value DB25_Male_MountingHoles (at 16.62 -18.44 180) (layer B.Fab)
+      (effects (font (size 1 1) (thickness 0.15)) (justify mirror))
+    )
+    (fp_text user %R (at 16.62 -13.94 180) (layer B.Fab)
+      (effects (font (size 1 1) (thickness 0.15)) (justify mirror))
+    )
+    (fp_line (start 43.7 2.35) (end -10.45 2.35) (layer B.CrtYd) (width 0.05))
+    (fp_line (start 43.7 -17.45) (end 43.7 2.35) (layer B.CrtYd) (width 0.05))
+    (fp_line (start -10.45 -17.45) (end 43.7 -17.45) (layer B.CrtYd) (width 0.05))
+    (fp_line (start -10.45 2.35) (end -10.45 -17.45) (layer B.CrtYd) (width 0.05))
+    (fp_line (start 0 2.321325) (end -0.25 2.754338) (layer B.SilkS) (width 0.12))
+    (fp_line (start 0.25 2.754338) (end 0 2.321325) (layer B.SilkS) (width 0.12))
+    (fp_line (start -0.25 2.754338) (end 0.25 2.754338) (layer B.SilkS) (width 0.12))
+    (fp_line (start 43.23 1.86) (end 43.23 -10.48) (layer B.SilkS) (width 0.12))
+    (fp_line (start -9.99 1.86) (end 43.23 1.86) (layer B.SilkS) (width 0.12))
+    (fp_line (start -9.99 -10.48) (end -9.99 1.86) (layer B.SilkS) (width 0.12))
+    (fp_line (start 41.77 -10.54) (end 41.77 -1.42) (layer B.Fab) (width 0.1))
+    (fp_line (start 38.57 -10.54) (end 38.57 -1.42) (layer B.Fab) (width 0.1))
+    (fp_line (start -5.33 -10.54) (end -5.33 -1.42) (layer B.Fab) (width 0.1))
+    (fp_line (start -8.53 -10.54) (end -8.53 -1.42) (layer B.Fab) (width 0.1))
+    (fp_line (start 42.67 -10.94) (end 37.67 -10.94) (layer B.Fab) (width 0.1))
+    (fp_line (start 42.67 -15.94) (end 42.67 -10.94) (layer B.Fab) (width 0.1))
+    (fp_line (start 37.67 -15.94) (end 42.67 -15.94) (layer B.Fab) (width 0.1))
+    (fp_line (start 37.67 -10.94) (end 37.67 -15.94) (layer B.Fab) (width 0.1))
+    (fp_line (start -4.43 -10.94) (end -9.43 -10.94) (layer B.Fab) (width 0.1))
+    (fp_line (start -4.43 -15.94) (end -4.43 -10.94) (layer B.Fab) (width 0.1))
+    (fp_line (start -9.43 -15.94) (end -4.43 -15.94) (layer B.Fab) (width 0.1))
+    (fp_line (start -9.43 -10.94) (end -9.43 -15.94) (layer B.Fab) (width 0.1))
+    (fp_line (start 35.77 -10.94) (end -2.53 -10.94) (layer B.Fab) (width 0.1))
+    (fp_line (start 35.77 -16.94) (end 35.77 -10.94) (layer B.Fab) (width 0.1))
+    (fp_line (start -2.53 -16.94) (end 35.77 -16.94) (layer B.Fab) (width 0.1))
+    (fp_line (start -2.53 -10.94) (end -2.53 -16.94) (layer B.Fab) (width 0.1))
+    (fp_line (start 43.17 -10.54) (end -9.93 -10.54) (layer B.Fab) (width 0.1))
+    (fp_line (start 43.17 -10.94) (end 43.17 -10.54) (layer B.Fab) (width 0.1))
+    (fp_line (start -9.93 -10.94) (end 43.17 -10.94) (layer B.Fab) (width 0.1))
+    (fp_line (start -9.93 -10.54) (end -9.93 -10.94) (layer B.Fab) (width 0.1))
+    (fp_line (start 43.17 1.8) (end -9.93 1.8) (layer B.Fab) (width 0.1))
+    (fp_line (start 43.17 -10.54) (end 43.17 1.8) (layer B.Fab) (width 0.1))
+    (fp_line (start -9.93 -10.54) (end 43.17 -10.54) (layer B.Fab) (width 0.1))
+    (fp_line (start -9.93 1.8) (end -9.93 -10.54) (layer B.Fab) (width 0.1))
+    (fp_arc (start 40.17 -1.42) (end 38.57 -1.42) (angle -180) (layer B.Fab) (width 0.1))
+    (fp_arc (start -6.93 -1.42) (end -8.53 -1.42) (angle -180) (layer B.Fab) (width 0.1))
+    (pad 0 thru_hole circle (at 40.17 -1.42 180) (size 4 4) (drill 3.2) (layers *.Cu *.Mask)
+      (net 58 "Net-(J3-Pad0)"))
+    (pad 0 thru_hole circle (at -6.93 -1.42 180) (size 4 4) (drill 3.2) (layers *.Cu *.Mask)
+      (net 58 "Net-(J3-Pad0)"))
+    (pad 25 thru_hole circle (at 31.855 -2.84 180) (size 1.6 1.6) (drill 1) (layers *.Cu *.Mask)
+      (net 9 /LPT_GND))
+    (pad 24 thru_hole circle (at 29.085 -2.84 180) (size 1.6 1.6) (drill 1) (layers *.Cu *.Mask)
+      (net 9 /LPT_GND))
+    (pad 23 thru_hole circle (at 26.315 -2.84 180) (size 1.6 1.6) (drill 1) (layers *.Cu *.Mask)
+      (net 9 /LPT_GND))
+    (pad 22 thru_hole circle (at 23.545 -2.84 180) (size 1.6 1.6) (drill 1) (layers *.Cu *.Mask)
+      (net 9 /LPT_GND))
+    (pad 21 thru_hole circle (at 20.775 -2.84 180) (size 1.6 1.6) (drill 1) (layers *.Cu *.Mask)
+      (net 9 /LPT_GND))
+    (pad 20 thru_hole circle (at 18.005 -2.84 180) (size 1.6 1.6) (drill 1) (layers *.Cu *.Mask)
+      (net 9 /LPT_GND))
+    (pad 19 thru_hole circle (at 15.235 -2.84 180) (size 1.6 1.6) (drill 1) (layers *.Cu *.Mask)
+      (net 9 /LPT_GND))
+    (pad 18 thru_hole circle (at 12.465 -2.84 180) (size 1.6 1.6) (drill 1) (layers *.Cu *.Mask)
+      (net 9 /LPT_GND))
+    (pad 17 thru_hole circle (at 9.695 -2.84 180) (size 1.6 1.6) (drill 1) (layers *.Cu *.Mask)
+      (net 59 "Net-(J3-Pad17)"))
+    (pad 16 thru_hole circle (at 6.925 -2.84 180) (size 1.6 1.6) (drill 1) (layers *.Cu *.Mask)
+      (net 60 "Net-(J3-Pad16)"))
+    (pad 15 thru_hole circle (at 4.155 -2.84 180) (size 1.6 1.6) (drill 1) (layers *.Cu *.Mask)
+      (net 61 "Net-(J3-Pad15)"))
+    (pad 14 thru_hole circle (at 1.385 -2.84 180) (size 1.6 1.6) (drill 1) (layers *.Cu *.Mask)
+      (net 62 "Net-(J3-Pad14)"))
+    (pad 13 thru_hole circle (at 33.24 0 180) (size 1.6 1.6) (drill 1) (layers *.Cu *.Mask)
+      (net 11 /EMERGENCY))
+    (pad 12 thru_hole circle (at 30.47 0 180) (size 1.6 1.6) (drill 1) (layers *.Cu *.Mask)
+      (net 12 /PROBE))
+    (pad 11 thru_hole circle (at 27.7 0 180) (size 1.6 1.6) (drill 1) (layers *.Cu *.Mask)
+      (net 63 "Net-(J3-Pad11)"))
+    (pad 10 thru_hole circle (at 24.93 0 180) (size 1.6 1.6) (drill 1) (layers *.Cu *.Mask)
+      (net 13 /SPINDLE_ENC))
+    (pad 9 thru_hole circle (at 22.16 0 180) (size 1.6 1.6) (drill 1) (layers *.Cu *.Mask)
+      (net 14 /SPINDLE_ENABLE))
+    (pad 8 thru_hole circle (at 19.39 0 180) (size 1.6 1.6) (drill 1) (layers *.Cu *.Mask)
+      (net 15 /SPINDLE_PWM))
+    (pad 7 thru_hole circle (at 16.62 0 180) (size 1.6 1.6) (drill 1) (layers *.Cu *.Mask)
+      (net 16 /AXIS_Z_STEP))
+    (pad 6 thru_hole circle (at 13.85 0 180) (size 1.6 1.6) (drill 1) (layers *.Cu *.Mask)
+      (net 17 /AXIS_Z_DIR))
+    (pad 5 thru_hole circle (at 11.08 0 180) (size 1.6 1.6) (drill 1) (layers *.Cu *.Mask)
+      (net 18 /AXIS_Y_STEP))
+    (pad 4 thru_hole circle (at 8.31 0 180) (size 1.6 1.6) (drill 1) (layers *.Cu *.Mask)
+      (net 19 /AXIS_Y_DIR))
+    (pad 3 thru_hole circle (at 5.54 0 180) (size 1.6 1.6) (drill 1) (layers *.Cu *.Mask)
+      (net 20 /AXIS_X_STEP))
+    (pad 2 thru_hole circle (at 2.77 0 180) (size 1.6 1.6) (drill 1) (layers *.Cu *.Mask)
+      (net 21 /AXIS_X_DIR))
+    (pad 1 thru_hole rect (at 0 0 180) (size 1.6 1.6) (drill 1) (layers *.Cu *.Mask)
+      (net 22 /ENABLE))
+    (model ${KISYS3DMOD}/Connector_Dsub.3dshapes/DSUB-25_Male_Horizontal_P2.77x2.84mm_EdgePinOffset7.70mm_Housed_MountingHolesOffset9.12mm.wrl
+      (at (xyz 0 0 0))
+      (scale (xyz 1 1 1))
+      (rotate (xyz 0 0 0))
+    )
+  )
   (module Relay_THT:Relay_SPDT_SANYOU_SRD_Series_Form_C (layer F.Cu)

Commit message: v4
Parts:
- D1, D2, K1, K2: moved to B.Cu
- moved J1 10.8 mm to (123.2, 38.7)
- moved D2 8.00 mm to (94.5, 37.5), turned to 270 degrees
- moved D1 7.01 mm to (54.0, 51.4), turned to 180 degrees
- moved H4 5.72 mm to (127.0, 29.8)
- moved R12 3.42 mm to (51.9, 54.6), turned to 0 degrees
- moved R11 1.46 mm to (51.9, 57.1), turned to 0 degrees
- moved K1 0.96 mm to (52.9, 41.7)
Routing:
- net VCC: track 92.7 -> 156.5 mm
- net Net-(D2-Pad2): track 105.3 -> 50.4 mm
- net Net-(J3-Pad0): track 0.00 -> 51.2 mm
- net Net-(D1-Pad1): track 11.5 -> 36.1 mm
- net Net-(D1-Pad2): track 102.2 -> 124.0 mm
- net Net-(D2-Pad1): track 10.8 -> 28.6 mm
- net Net-(J6-Pad3): track 7.83 -> 23.8 mm
- net GND: track 137.7 -> 150.1 mm
- net Net-(J5-Pad1): track 9.55 -> 20.4 mm
- net /LPT_GND: track 212.3 -> 206.1 mm
- net Net-(J4-Pad2): track 38.5 -> 43.3 mm
- net /EMERGENCY: track 28.7 -> 31.4 mm
- net Net-(J6-Pad4): track 20.1 -> 17.7 mm
- net Net-(R11-Pad2): track 2.86 -> 4.53 mm
- net Net-(J7-Pad2): track 34.4 -> 36.0 mm
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Other:
- net class Default: trace_width 0.4 -> 0.6; via_dia 1.2 -> 1.4
- net class pwr: via_dia 1.2 -> 1.4
- rule trace_min: 0.2 -> 0.6
