File: cncshitter/cncshitter.kicad_pcb (KiCad board)
At the start: 2 copper layers, 104 x 70 mm, 54 parts, among them J1 24V_IN, J2 5V_IN, J3 DB25_Male_MountingHoles, J4 SPINDLE_PWM_ENC, J5 SPINDLE_ENABLE, J6 EMERGENCY_PROBE_ENABLE, J7 AXIS_XYZ, K1 SANYOU_SRD_Form_C, K2 SANYOU_SRD_Form_C, U1 EMERGENCY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

Commit message: v5
Parts:
- added Q1: BC847, Package_TO_SOT_SMD:SOT-23, F.Cu at (68.8, 73.2)
- added Q2: BC847, Package_TO_SOT_SMD:SOT-23, F.Cu at (59.9, 73.2)
- added Q3: BC847, Package_TO_SOT_SMD:SOT-23, F.Cu at (128.8, 73.2)
- added Q4: BC847, Package_TO_SOT_SMD:SOT-23, F.Cu at (120.4, 73.2)
- added Q5: BC847, Package_TO_SOT_SMD:SOT-23, F.Cu at (112.0, 73.2)
- added Q6: BC847, Package_TO_SOT_SMD:SOT-23, F.Cu at (103.6, 73.2)
- added Q7: BC847, Package_TO_SOT_SMD:SOT-23, F.Cu at (95.2, 73.1)
- added Q8: BC847, Package_TO_SOT_SMD:SOT-23, F.Cu at (86.7, 73.1)
- added Q9: BC847, Package_TO_SOT_SMD:SOT-23, F.Cu at (77.7, 73.1)
- added R26: 6k8, Resistor_SMD:R_1206_3216Metric_Pad1.42x1.75mm_HandSolder, F.Cu at (119.1, 77.8)
- added R27: 6k8, Resistor_SMD:R_1206_3216Metric_Pad1.42x1.75mm_HandSolder, F.Cu at (110.7, 77.8)
- added R28: 6k8, Resistor_SMD:R_1206_3216Metric_Pad1.42x1.75mm_HandSolder, F.Cu at (102.4, 77.8)
- added R29: 6k8, Resistor_SMD:R_1206_3216Metric_Pad1.42x1.75mm_HandSolder, F.Cu at (94.0, 77.7)
- added R30: 6k8, Resistor_SMD:R_1206_3216Metric_Pad1.42x1.75mm_HandSolder, F.Cu at (85.3, 77.8)
- added R31: 6k8, Resistor_SMD:R_1206_3216Metric_Pad1.42x1.75mm_HandSolder, F.Cu at (76.5, 77.8)
- added R32: 680R, Resistor_SMD:R_1206_3216Metric_Pad1.42x1.75mm_HandSolder, F.Cu at (121.7, 77.8)
- added R33: 680R, Resistor_SMD:R_1206_3216Metric_Pad1.42x1.75mm_HandSolder, F.Cu at (113.3, 77.8)
- added R34: 680R, Resistor_SMD:R_1206_3216Metric_Pad1.42x1.75mm_HandSolder, F.Cu at (104.9, 77.8)
- added R35: 680R, Resistor_SMD:R_1206_3216Metric_Pad1.42x1.75mm_HandSolder, F.Cu at (96.5, 77.7)
- added R36: 680R, Resistor_SMD:R_1206_3216Metric_Pad1.42x1.75mm_HandSolder, F.Cu at (87.9, 77.7)
- added R37: 680R, Resistor_SMD:R_1206_3216Metric_Pad1.42x1.75mm_HandSolder, F.Cu at (79.0, 77.7)
- added R38: 680R, Resistor_SMD:R_1206_3216Metric_Pad1.42x1.75mm_HandSolder, F.Cu at (116.6, 74.7)
- added R39: 680R, Resistor_SMD:R_1206_3216Metric_Pad1.42x1.75mm_HandSolder, F.Cu at (108.2, 74.7)
- added R40: 680R, Resistor_SMD:R_1206_3216Metric_Pad1.42x1.75mm_HandSolder, F.Cu at (99.8, 74.7)
- added R41: 680R, Resistor_SMD:R_1206_3216Metric_Pad1.42x1.75mm_HandSolder, F.Cu at (91.4, 74.7)
- added R42: 680R, Resistor_SMD:R_1206_3216Metric_Pad1.42x1.75mm_HandSolder, F.Cu at (82.8, 74.7)
- added R43: 680R, Resistor_SMD:R_1206_3216Metric_Pad1.42x1.75mm_HandSolder, F.Cu at (73.9, 74.7)
- R14, R15, R16, R17, R19, R3: value 1k -> 680R
- R18, R4, R6: value 1k -> 6k8
- moved J2 69.1 mm to (48.0, 85.3)
- moved R19 54.5 mm to (129.8, 77.7)
- moved R15 48.6 mm to (61.2, 77.7)
- moved R14 47.4 mm to (70.1, 77.7)
- moved R18 43.1 mm to (127.3, 77.7)
- moved R17 38.5 mm to (54.9, 71.4)
- moved R16 37.1 mm to (65.0, 74.7)
- moved J3 23.2 mm to (111.9, 86.7)
- moved R1 9.16 mm to (41.9, 78.7), turned to 270 degrees
- moved R5 4.83 mm to (52.1, 78.7), turned to 270 degrees
- moved R4 3.65 mm to (67.6, 77.8)
- moved R6 3.58 mm to (58.7, 77.7)
- moved R2 2.93 mm to (44.5, 75.7)
- moved R9 2.81 mm to (37.1, 56.1)
- moved U1 2.54 mm to (35.6, 64.8)
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Connections:
- J2 pad 1: /LPT_GND -> /LPT_VCC
- J2 pad 2: /LPT_VCC -> /LPT_GND
- R14 pad 1: /AXIS_X_DIR -> /LPT_VCC
- R14 pad 2: Net-(R14-Pad2) -> Net-(Q1-Pad3)
- R15 pad 1: /AXIS_X_STEP -> /LPT_VCC
- R15 pad 2: Net-(R15-Pad2) -> Net-(Q2-Pad3)
- R16 pad 1: /AXIS_Y_DIR -> /LPT_VCC
- R17 pad 1: /AXIS_Y_STEP -> /LPT_VCC
- R18 pad 1: /AXIS_Z_DIR -> /ENABLE
- R18 pad 2: Net-(R18-Pad2) -> Net-(Q3-Pad1)
- R19 pad 1: /AXIS_Z_STEP -> /LPT_VCC
- R19 pad 2: Net-(R19-Pad2) -> Net-(Q3-Pad3)
- R3 pad 1: /ENABLE -> /LPT_VCC
- R4 pad 2: Net-(R4-Pad2) -> Net-(Q1-Pad1)
- R6 pad 2: Net-(R6-Pad2) -> Net-(Q2-Pad1)
- U10 pad 1: Net-(R17-Pad2) -> Net-(R41-Pad2)
- U10 pad 2: /LPT_GND -> Net-(Q7-Pad3)
- U11 pad 1: Net-(R18-Pad2) -> Net-(R42-Pad2)
- U11 pad 2: /LPT_GND -> Net-(Q8-Pad3)
- U12 pad 1: Net-(R19-Pad2) -> Net-(R43-Pad2)
- U12 pad 2: /LPT_GND -> Net-(Q9-Pad3)
- U3 pad 2: /LPT_GND -> Net-(Q3-Pad3)
- U4 pad 1: Net-(R4-Pad2) -> Net-(R16-Pad2)
- U4 pad 2: /LPT_GND -> Net-(Q1-Pad3)
- U6 pad 1: Net-(R6-Pad2) -> Net-(R17-Pad2)
- U6 pad 2: /LPT_GND -> Net-(Q2-Pad3)
- U7 pad 1: Net-(R14-Pad2) -> Net-(R38-Pad2)
- U7 pad 2: /LPT_GND -> Net-(Q4-Pad3)
- U8 pad 1: Net-(R15-Pad2) -> Net-(R39-Pad2)
- U8 pad 2: /LPT_GND -> Net-(Q5-Pad3)
- U9 pad 1: Net-(R16-Pad2) -> Net-(R40-Pad2)
- U9 pad 2: /LPT_GND -> Net-(Q6-Pad3)
Routing:
- net /LPT_GND: track 206.1 -> 256.3 mm
- net /LPT_VCC: track 104.6 -> 137.3 mm, vias 4 -> 2
- net /SPINDLE_ENC: track 20.4 -> 50.5 mm
- net /EMERGENCY: track 31.4 -> 60.4 mm
- net /PROBE: track 24.7 -> 49.4 mm
- net /AXIS_X_DIR: track 34.6 -> 13.0 mm
- net /SPINDLE_ENABLE: track 13.9 -> 35.0 mm
- net /ENABLE: track 39.4 -> 18.4 mm
- net /AXIS_X_STEP: track 29.7 -> 9.27 mm
- net /SPINDLE_PWM: track 9.30 -> 28.1 mm
- net /AXIS_Y_DIR: track 24.9 -> 8.00 mm
- net /AXIS_Z_STEP: track 9.38 -> 22.4 mm
- net Net-(Q6-Pad3): track 0.00 -> 7.50 mm
- net Net-(Q4-Pad3): track 0.00 -> 7.35 mm
- net Net-(Q5-Pad3): track 0.00 -> 7.05 mm
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