File: cncshitter/cncshitter.kicad_pcb (KiCad board)
At the start: 2 copper layers, 104 x 70 mm, 81 parts, among them J1 24V_IN, J2 5V_IN, J3 DB25_Male_MountingHoles, J4 SPINDLE_PWM_ENC, J5 SPINDLE_ENABLE, J6 EMERGENCY_PROBE_ENABLE, J7 AXIS_XYZ, K1 SANYOU_SRD_Form_C, K2 SANYOU_SRD_Form_C, Q1 BC847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

Commit message: v6
Parts:
- added H2: MountingHole, MountingHole:MountingHole_3mm_Pad, F.Cu at (67.1, 37.6)
- moved R13 19.7 mm to (101.6, 37.1), turned to 180 degrees
- moved R7 7.99 mm to (72.1, 45.8)
- moved C1 7.51 mm to (65.4, 44.7)
- moved C2 6.62 mm to (65.4, 47.6)
- moved C3 5.48 mm to (65.4, 50.3)
- moved R8 5.15 mm to (69.6, 48.7)
- moved D2 3.05 mm to (97.5, 37.5)
- moved K2 2.03 mm to (92.7, 41.7)
- moved R23 1.53 mm to (94.7, 56.4), turned to 180 degrees
- moved R24 1.53 mm to (85.8, 56.4), turned to 180 degrees
- moved J1 1.14 mm to (123.2, 37.6)
Connections:
- net Net-(J5-Pad1) renamed /HV_SPINDLE_EN_A
- net Net-(J5-Pad2) renamed /HV_SPINDLE_EN_B
- net Net-(J6-Pad3) renamed /HV_ENABLE_A
- net Net-(J6-Pad4) renamed /HV_ENABLE_B
Routing:
- net VCC: track 153.5 -> 133.9 mm
- net Net-(D2-Pad1): track 28.6 -> 11.2 mm
- net Net-(C1-Pad1): track 20.0 -> 27.8 mm
- net Net-(J4-Pad5): track 9.93 -> 16.2 mm
- net Net-(R7-Pad1): track 26.8 -> 20.7 mm
- net Net-(J7-Pad3): track 29.3 -> 34.5 mm
- net /HV_SPINDLE_EN_B: track 20.6 -> 16.9 mm
- net /HV_ENABLE_A: track 23.8 -> 20.3 mm
- net Net-(J7-Pad4): track 27.7 -> 30.2 mm
- net Net-(J7-Pad1): track 48.5 -> 46.1 mm
- net Net-(J7-Pad2): track 36.0 -> 37.5 mm
- net Net-(C1-Pad2): track 34.1 -> 35.5 mm
- net Net-(R23-Pad2): track 2.86 -> 4.10 mm
- net Net-(R24-Pad2): track 2.86 -> 4.00 mm
- net GND: track 152.5 -> 153.6 mm
Other:
- net class hv added: clearance 1.3, trace_width 1, via_dia 1.4, via_drill 1

Commit message: v7
Parts:
- removed J6: EMERGENCY_PROBE_ENABLE, Connector_Phoenix_MC_HighVoltage:PhoenixContact_MC_1,5_4-G-5.08_1x04_P5.08mm_Horizontal
- removed J7: AXIS_XYZ, Connector_Phoenix_MC_HighVoltage:PhoenixContact_MC_1,5_6-G-5.08_1x06_P5.08mm_Horizontal
- J1, J2: footprint Connector_Phoenix_MC_HighVoltage:PhoenixContact_MC_1,5_2-G-5.08_1x02_P5.08mm_Horizontal -> Connector_Phoenix_MC_HighVoltage:PhoenixContact_MCV_1,5_2-G-5.08_1x02_P5.08mm_Vertical
- J4: value SPINDLE_PWM_ENC -> Screw_Terminal_01x11; footprint Connector_Phoenix_MC_HighVoltage:PhoenixContact_MC_1,5_5-G-5.08_1x05_P5.08mm_Horizontal -> Connector_Phoenix_MC_HighVoltage:PhoenixContact_MCV_1,5_11-G-5.08_1x11_P5.08mm_Vertical
- J5: value SPINDLE_ENABLE -> Screw_Terminal_01x06; footprint Connector_Phoenix_MC_HighVoltage:PhoenixContact_MC_1,5_2-G-5.08_1x02_P5.08mm_Horizontal -> Connector_Phoenix_MC_HighVoltage:PhoenixContact_MCV_1,5_6-G-5.08_1x06_P5.08mm_Vertical
- moved J5 48.0 mm to (32.5, 29.5)
- moved D1 11.6 mm to (56.4, 40.1), turned to 270 degrees
- moved J4 10.2 mm to (64.0, 29.5)
- moved J1 4.49 mm to (126.5, 40.6)
- moved K1 2.91 mm to (51.2, 44.0)
- moved K2 2.08 mm to (92.7, 43.7)
- moved H2 1.02 mm to (67.1, 38.6)
Connections:
- C1 pad 1: Net-(C1-Pad1) -> /PWM_B
- C1 pad 2: Net-(C1-Pad2) -> /PWM_C
- C2 pad 1: Net-(C1-Pad1) -> /PWM_B
- C2 pad 2: Net-(C1-Pad2) -> /PWM_C
- C3 pad 1: Net-(C1-Pad1) -> /PWM_B
- C3 pad 2: Net-(C1-Pad2) -> /PWM_C
- J4 pad 1: GND -> /PWM_C
- J4 pad 2: Net-(J4-Pad2) -> /PWM_B
- J4 pad 3: Net-(C1-Pad2) -> /PWM_A
- J4 pad 4: Net-(C1-Pad1) -> /HV_SPINDLE_EN_A
- J4 pad 5: Net-(J4-Pad5) -> /HV_SPINDLE_EN_B
- J5 pad 1: /HV_SPINDLE_EN_A -> Net-(J5-Pad1)
- J5 pad 2: /HV_SPINDLE_EN_B -> Net-(J5-Pad2)
- R20 pad 1: Net-(J7-Pad6) -> /X_DIR
- R21 pad 1: Net-(J7-Pad5) -> /X_STEP
- R22 pad 1: Net-(J7-Pad4) -> /Y_DIR
- R23 pad 1: Net-(J7-Pad3) -> /Y_STEP
- R24 pad 1: Net-(J7-Pad2) -> /Z_DIR
- R25 pad 1: Net-(J7-Pad1) -> /Z_STEP
- R7 pad 2: Net-(J4-Pad5) -> /PWM_A
- R8 pad 1: Net-(C1-Pad1) -> /PWM_B
- U1 pad 2: Net-(J6-Pad1) -> Net-(J5-Pad1)
- U2 pad 2: Net-(J6-Pad2) -> Net-(J5-Pad2)
- U4 pad 3: Net-(C1-Pad2) -> /PWM_C
- U5 pad 2: Net-(J4-Pad2) -> /ENC
Routing:
- net Net-(J7-Pad1): track 46.1 -> 0.00 mm
- net /Z_STEP: track 0.00 -> 46.0 mm
- net /ENC: track 0.00 -> 44.4 mm
- net Net-(J4-Pad2): track 43.0 -> 0.00 mm
- net Net-(J5-Pad2): track 0.00 -> 42.9 mm
- net Net-(J6-Pad2): track 41.7 -> 0.00 mm
- net /Z_DIR: track 0.00 -> 39.9 mm
- net Net-(J7-Pad2): track 37.5 -> 0.00 mm
- net /Y_STEP: track 0.00 -> 36.2 mm
- net Net-(D1-Pad2): track 124.7 -> 88.9 mm
- net /PWM_C: track 0.00 -> 35.6 mm
- net Net-(C1-Pad2): track 35.5 -> 0.00 mm
- net Net-(J7-Pad3): track 34.5 -> 0.00 mm
- net Net-(J5-Pad1): track 0.00 -> 34.3 mm
- net Net-(J6-Pad1): track 34.1 -> 0.00 mm
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
Commit message: v8
Parts:
- moved R13 0.51 mm to (101.6, 37.6)
Routing:
- net /ENC: track 44.4 -> 42.1 mm
- net /Y_STEP: track 36.2 -> 34.5 mm
- net /Y_DIR: track 32.3 -> 30.8 mm
- net /Z_DIR: track 39.9 -> 38.6 mm
- net Net-(D1-Pad1): track 31.5 -> 30.3 mm
- net /LPT_VCC: track 137.3 -> 136.5 mm
- net Net-(D1-Pad2): track 88.9 -> 89.5 mm

Commit message: vkkt
Parts:
- moved J3 12.1 mm to (99.8, 86.1)
- moved H1 3.18 mm to (33.0, 88.0)
- moved H3 2.92 mm to (127.3, 88.0)
- moved H4 0.31 mm to (127.3, 30.0)
Routing:
- net /PROBE: track 49.4 -> 36.3 mm
- net /SPINDLE_ENABLE: track 35.0 -> 22.5 mm
- net /SPINDLE_ENC: track 50.5 -> 38.1 mm
- net /EMERGENCY: track 60.5 -> 48.3 mm
- net /LPT_GND: track 256.3 -> 244.3 mm
- net /SPINDLE_PWM: track 28.1 -> 16.2 mm
- net /ENABLE: track 18.4 -> 30.3 mm
- net /AXIS_X_DIR: track 13.0 -> 24.9 mm
- net /AXIS_Z_STEP: track 22.4 -> 10.9 mm
- net /AXIS_X_STEP: track 9.27 -> 19.3 mm
- net /AXIS_Z_DIR: track 15.9 -> 7.25 mm
- net /AXIS_Y_DIR: track 8.00 -> 14.4 mm
- net /AXIS_Y_STEP: track 12.0 -> 9.89 mm
- net Net-(J3-Pad0): track 52.3 -> 50.6 mm
