File: cncshitter/cncshitter.sch (KiCad schematic (older format))
At the start: 51 parts, among them J1 24V_IN, J2 5V_IN, J3 DB25_Male_MountingHoles, J4 SPINDLE_PWM_ENC, J5 SPINDLE_ENABLE, J6 EMERGENCY_PROBE_ENABLE, J7 AXIS_XYZ, K1 SANYOU_SRD_Form_C, K2 SANYOU_SRD_Form_C, U1 EMERGENCY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

Commit message: v2
Parts:
- added H1, H2, H3, H4: MountingHole, MountingHole:MountingHole_3mm_Pad, symbol Mechanical:MountingHole
Connections:
- net GND: now also J4.1 (Pin_1); no longer J4.5 (Pin_5)
- net LPT_GND: now also U4.2
- net at C1.1, C2.1, C3.1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: now also J4.4 (Pin_4); no longer J4.2 (Pin_2)
- net at R7.2: now also J4.5 (Pin_5); no longer J4.1 (Pin_1)
- net at U5.2: now also J4.2 (Pin_2); no longer J4.4 (Pin_4)
Changed lines of the file:
@@
 EESchema Schematic File Version 4
+LIBS:cncshitter-cache
 EELAYER 29 0
 EELAYER END
@@
 F 3 "~" H 6050 4650 50  0001 C CNN
 	1    6050 4650
-	1    0    0    -1
+	1    0    0    1
 $EndComp
 $Comp
@@
 Wire Wire Line
 	3900 4200 4050 4200
-Text Label 3800 4300 0    50   ~ 0
+Text Label 3900 4200 2    50   ~ 0
 LPT_GND
 Wire Wire Line
@@
 Text Label 1900 3350 0    50   ~ 0
 SPINDLE_ENABLE
+$Comp
+L Mechanical:MountingHole H1
+U 1 1 5E20C0CA
+P 1550 5900
+F 0 "H1" H 1650 5946 50  0000 L CNN
+F 1 "MountingHole" H 1650 5855 50  0000 L CNN
+F 2 "MountingHole:MountingHole_3mm_Pad" H 1550 5900 50  0001 C CNN
+F 3 "~" H 1550 5900 50  0001 C CNN
+	1    1550 5900
+	1    0    0    -1
+$EndComp
+$Comp
+L Mechanical:MountingHole H2
+U 1 1 5E20C43C
+P 1550 6100
+F 0 "H2" H 1650 6146 50  0000 L CNN
+F 1 "MountingHole" H 1650 6055 50  0000 L CNN
+F 2 "MountingHole:MountingHole_3mm_Pad" H 1550 6100 50  0001 C CNN
+F 3 "~" H 1550 6100 50  0001 C CNN
+	1    1550 6100
+	1    0    0    -1
+$EndComp
+$Comp
+L Mechanical:MountingHole H3
+U 1 1 5E20C642
+P 1550 6300
+F 0 "H3" H 1650 6346 50  0000 L CNN
+F 1 "MountingHole" H 1650 6255 50  0000 L CNN
+F 2 "MountingHole:MountingHole_3mm_Pad" H 1550 6300 50  0001 C CNN
+F 3 "~" H 1550 6300 50  0001 C CNN
+	1    1550 6300
+	1    0    0    -1
+$EndComp
+$Comp
+L Mechanical:MountingHole H4
+U 1 1 5E20C81F
+P 1550 6500
+F 0 "H4" H 1650 6546 50  0000 L CNN
+F 1 "MountingHole" H 1650 6455 50  0000 L CNN
+F 2 "MountingHole:MountingHole_3mm_Pad" H 1550 6500 50  0001 C CNN
+F 3 "~" H 1550 6500 50  0001 C CNN
+	1    1550 6500
+	1    0    0    -1
+$EndComp
 $EndSCHEMATC

Commit message: v3 smaller
Parts:
- removed H2: MountingHole, MountingHole:MountingHole_3mm_Pad, symbol Mechanical:MountingHole
Changed lines of the file:
@@
 SPINDLE_ENABLE
+$Comp
+L Mechanical:MountingHole H3
+U 1 1 5E20C642
+P 1550 6300
+F 0 "H3" H 1650 6346 50  0000 L CNN
+F 1 "MountingHole" H 1650 6255 50  0000 L CNN
+F 2 "MountingHole:MountingHole_3mm_Pad" H 1550 6300 50  0001 C CNN
+F 3 "~" H 1550 6300 50  0001 C CNN
+	1    1550 6300
+	1    0    0    -1
+$EndComp
 $Comp
 L Mechanical:MountingHole H1
@@
 	1    0    0    -1
 $EndComp
-$Comp
-L Mechanical:MountingHole H2
-U 1 1 5E20C43C
-P 1550 6100
-F 0 "H2" H 1650 6146 50  0000 L CNN
-F 1 "MountingHole" H 1650 6055 50  0000 L CNN
-F 2 "MountingHole:MountingHole_3mm_Pad" H 1550 6100 50  0001 C CNN
-F 3 "~" H 1550 6100 50  0001 C CNN
-	1    1550 6100
-	1    0    0    -1
-$EndComp
-$Comp
-L Mechanical:MountingHole H3
-U 1 1 5E20C642
-P 1550 6300
-F 0 "H3" H 1650 6346 50  0000 L CNN
-F 1 "MountingHole" H 1650 6255 50  0000 L CNN
-F 2 "MountingHole:MountingHole_3mm_Pad" H 1550 6300 50  0001 C CNN
-F 3 "~" H 1550 6300 50  0001 C CNN
-	1    1550 6300
-	1    0    0    -1
-$EndComp

Commit message: v5
Parts:
- removed R14, R15, R19: 1k, Resistor_SMD:R_1206_3216Metric_Pad1.42x1.75mm_HandSolder, symbol Device:R
- added Q1, Q2, Q3, Q4, Q5, Q6, Q7, Q8, Q9: BC847, Package_TO_SOT_SMD:SOT-23, symbol Transistor_BJT:BC847
- added R26, R27, R28, R29, R30, R31: 6k8, Resistor_SMD:R_1206_3216Metric_Pad1.42x1.75mm_HandSolder, symbol Device:R
- added R38, R39, R40, R41, R42, R43: 680R, Resistor_SMD:R_1206_3216Metric_Pad1.42x1.75mm_HandSolder, symbol Device:R
- R16, R17, R3: value 1k -> 680R
- R18, R4, R6: value 1k -> 6k8
Connections:
- net AXIS_X_DIR: now also R26.1
- net AXIS_X_STEP: now also R27.1
- net AXIS_Y_DIR: now also R28.1; no longer R16.1
- net AXIS_Y_STEP: now also R29.1; no longer R17.1
- net AXIS_Z_DIR: now also R30.1; no longer R18.1
- net AXIS_Z_STEP: now also R31.1
- net ENABLE: now also R18.1; no longer R3.1
- net LPT_GND: now also J2.2 (Pin_2), Q1.2 (E), Q2.2 (E), Q3.2 (E), Q4.2 (E), Q5.2 (E), Q6.2 (E), Q7.2 (E), Q8.2 (E), Q9.2 (E); no longer J2.1 (Pin_1), U10.2, U11.2, U12.2, U3.2, U4.2, U6.2, U7.2, U8.2, U9.2
- net LPT_VCC: now also J2.1 (Pin_1), R16.1, R17.1, R3.1, R38.1, R39.1, R40.1, R41.1, R42.1, R43.1; no longer J2.2 (Pin_2)
- net at U7.1: now also R38.2
- net at U8.1: now also R39.2
- net at U9.1: now also R40.2; no longer R16.2
- net at U10.1: now also R41.2; no longer R17.2
- net at U11.1: now also R42.2; no longer R18.2
- net at U12.1: now also R43.2
- net at U4.1: now also R16.2; no longer R4.2
- net at U6.1: now also R17.2; no longer R6.2
- new net: Q4.3 (C), U7.2
- new net: Q5.3 (C), U8.2
- new net: Q6.3 (C), U9.2
- new net: Q7.3 (C), U10.2
- new net: Q8.3 (C), U11.2
- new net: Q9.3 (C), U12.2
- new net: Q3.1 (B), R18.2
- new net: Q3.3 (C), U3.2
- new net: Q1.3 (C), U4.2
- new net: Q1.1 (B), R4.2
- new net: Q2.3 (C), U6.2
- new net: Q2.1 (B), R6.2
- new net: Q4.1 (B), R26.2
- new net: Q5.1 (B), R27.2
- new net: Q6.1 (B), R28.2
- new net: Q8.1 (B), R30.2
- new net: Q7.1 (B), R29.2
- new net: Q9.1 (B), R31.2
Other:
- moved on the sheet: C1, C2, C3, D1, D2, H1, H3, H4, J1, J2, J3, J4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

Commit message: v6
Parts:
- added H2: MountingHole, MountingHole:MountingHole_3mm_Pad, symbol Mechanical:MountingHole
Connections:
- net HV_SPINDLE_EN_B: now reaches J5.2 (Pin_2), K2.1
- net HV_SPINDLE_EN_A: now reaches J5.1 (Pin_1), K2.3
- net HV_ENABLE_B: now reaches J6.4 (Pin_4), K1.1
- net HV_ENABLE_A: now reaches J6.3 (Pin_3), K1.3
Other:
- moved on the sheet: J5
Changed lines of the file:
@@
 L Connector:Screw_Terminal_01x02 J5
 U 1 1 5E250E9A
-P 4600 7150
-F 0 "J5" H 4680 7142 50  0000 L CNN
-F 1 "SPINDLE_ENABLE" H 4680 7051 50  0000 L CNN
-F 2 "Connector_Phoenix_MC_HighVoltage:PhoenixContact_MC_1,5_2-G-5.08_1x02_P5.08mm_Horizontal" H 4600 7150 50  0001 C CNN
-F 3 "~" H 4600 7150 50  0001 C CNN
-	1    4600 7150
-	1    0    0    -1
-$EndComp
-Wire Wire Line
-	4150 7150 4400 7150
-Wire Wire Line
-	4400 7250 4400 7350
-Wire Wire Line
-	4400 7350 3550 7350
+P 5050 7150
+F 0 "J5" H 5130 7142 50  0000 L CNN
+F 1 "SPINDLE_ENABLE" H 5130 7051 50  0000 L CNN
+F 2 "Connector_Phoenix_MC_HighVoltage:PhoenixContact_MC_1,5_2-G-5.08_1x02_P5.08mm_Horizontal" H 5050 7150 50  0001 C CNN
+F 3 "~" H 5050 7150 50  0001 C CNN
+	1    5050 7150
+	1    0    0    -1
+$EndComp
 Wire Wire Line
 	3550 7350 3550 7050
@@
 Wire Wire Line
 	2100 6850 2600 6850
+Text Label 5350 3300 0    50   ~ 0
+HV_ENABLE_A
+Text Label 5350 3500 0    50   ~ 0
+HV_ENABLE_B
+Wire Wire Line
+	4150 7150 4850 7150
+Wire Wire Line
+	4800 7350 4800 7250
+Wire Wire Line
+	4800 7250 4850 7250
+Wire Wire Line
+	3550 7350 4800 7350
+Text Label 4100 7350 0    50   ~ 0
+HV_SPINDLE_EN_B
+Text Label 4200 7150 0    50   ~ 0
+HV_SPINDLE_EN_A
+$Comp
+L Mechanical:MountingHole H2
+U 1 1 5E711BB7
+P 6000 4650
+F 0 "H2" H 6100 4696 50  0000 L CNN
+F 1 "MountingHole" H 6100 4605 50  0000 L CNN
+F 2 "MountingHole:MountingHole_3mm_Pad" H 6000 4650 50  0001 C CNN
+F 3 "~" H 6000 4650 50  0001 C CNN
+	1    6000 4650
+	1    0    0    -1
+$EndComp
 $EndSCHEMATC

Commit message: v7
Parts:
- removed J4: SPINDLE_PWM_ENC, Connector_Phoenix_MC_HighVoltage:PhoenixContact_MC_1,5_5-G-5.08_1x05_P5.08mm_Horizontal, symbol Connector:Screw_Terminal_01x05
- removed J5: SPINDLE_ENABLE, Connector_Phoenix_MC_HighVoltage:PhoenixContact_MC_1,5_2-G-5.08_1x02_P5.08mm_Horizontal, symbol Connector:Screw_Terminal_01x02
- removed J6: EMERGENCY_PROBE_ENABLE, Connector_Phoenix_MC_HighVoltage:PhoenixContact_MC_1,5_4-G-5.08_1x04_P5.08mm_Horizontal, symbol Connector:Screw_Terminal_01x04
- removed J7: AXIS_XYZ, Connector_Phoenix_MC_HighVoltage:PhoenixContact_MC_1,5_6-G-5.08_1x06_P5.08mm_Horizontal, symbol Connector:Screw_Terminal_01x06
- added J4: Screw_Terminal_01x11, Connector_Phoenix_MC_HighVoltage:PhoenixContact_MCV_1,5_11-G-5.08_1x11_P5.08mm_Vertical, symbol Connector:Screw_Terminal_01x11
- added J5: Screw_Terminal_01x06, Connector_Phoenix_MC_HighVoltage:PhoenixContact_MCV_1,5_6-G-5.08_1x06_P5.08mm_Vertical, symbol Connector:Screw_Terminal_01x06
- J1, J2: footprint Connector_Phoenix_MC_HighVoltage:PhoenixContact_MC_1,5_2-G-5.08_1x02_P5.08mm_Horizontal -> Connector_Phoenix_MC_HighVoltage:PhoenixContact_MCV_1,5_2-G-5.08_1x02_P5.08mm_Vertical
Connections:
- net GND: now also J5.5 (Pin_5)
- net HV_ENABLE_A: now also J5.3 (Pin_3)
- net HV_ENABLE_B: now also J5.4 (Pin_4)
- net HV_SPINDLE_EN_A: now also J4.4 (Pin_4)
- net HV_SPINDLE_EN_B: now also J4.5 (Pin_5)
- net Z_STEP: now reaches R25.1
- net Z_STEP: now also J4.6 (Pin_6)
- net Z_DIR: now reaches R24.1
- net Z_DIR: now also J4.7 (Pin_7)
- net Y_STEP: now reaches R23.1
- net Y_STEP: now also J4.8 (Pin_8)
- net Y_DIR: now reaches R22.1
- net Y_DIR: now also J4.9 (Pin_9)
- net X_STEP: now reaches R21.1
- net X_STEP: now also J4.10 (Pin_10)
- net X_DIR: now reaches R20.1
- net X_DIR: now also J4.11 (Pin_11)
- net at U1.2: now also J5.1 (Pin_1)
- net at U2.2: now also J5.2 (Pin_2)
- net PWM_C: now reaches C1.2, C2.2, C3.2, U4.3
- net PWM_C: now also J4.1 (Pin_1)
- net PWM_B: now reaches C1.1, C2.1, C3.1, R8.1
- net PWM_B: now also J4.2 (Pin_2)
- net PWM_A: now reaches R7.2
- net PWM_A: now also J4.3 (Pin_3)
- net ENC: now reaches U5.2
- net ENC: now also J5.6 (Pin_6)
Changed lines of the file:
@@
-$EndComp
-$Comp
-L Connector:Screw_Terminal_01x06 J7
-U 1 1 5E191CCA
-P 10950 3400
-F 0 "J7" H 10868 2875 50  0000 C CNN
-F 1 "AXIS_XYZ" H 10868 2966 50  0000 C CNN
-F 2 "Connector_Phoenix_MC_HighVoltage:PhoenixContact_MC_1,5_6-G-5.08_1x06_P5.08mm_Horizontal" H 10950 3400 50  0001 C CNN
-F 3 "~" H 10950 3400 50  0001 C CNN
-	1    10950 3400
-	1    0    0    1
 $EndComp
 $Comp
@@
 F 0 "J1" H 6230 5492 50  0000 L CNN
 F 1 "24V_IN" H 6230 5401 50  0000 L CNN
-F 2 "Connector_Phoenix_MC_HighVoltage:PhoenixContact_MC_1,5_2-G-5.08_1x02_P5.08mm_Horizontal" H 6150 5500 50  0001 C CNN
+F 2 "Connector_Phoenix_MC_HighVoltage:PhoenixContact_MCV_1,5_2-G-5.08_1x02_P5.08mm_Vertical" H 6150 5500 50  0001 C CNN
 F 3 "~" H 6150 5500 50  0001 C CNN
 	1    6150 5500
@@
 	5100 1850 5200 1850
 Wire Wire Line
-	3200 5800 4400 5800
-Wire Wire Line
 	4150 5250 4150 5700
 Wire Wire Line
-	4150 5700 4400 5700
-Wire Wire Line
 	4000 5250 4150 5250
 Wire Wire Line
 	4300 4900 4300 5600
-Wire Wire Line
-	4300 5600 4400 5600
 Wire Wire Line
 	4000 4900 4200 4900
@@
 Wire Wire Line
 	3400 6650 3550 6650
-$Comp
-L Connector:Screw_Terminal_01x05 J4
-U 1 1 5E21A47A
-P 4600 5700
-F 0 "J4" H 4680 5742 50  0000 L CNN
-F 1 "SPINDLE_PWM_ENC" H 4680 5651 50  0000 L CNN
-F 2 "Connector_Phoenix_MC_HighVoltage:PhoenixContact_MC_1,5_5-G-5.08_1x05_P5.08mm_Horizontal" H 4600 5700 50  0001 C CNN
-F 3 "~" H 4600 5700 50  0001 C CNN
-	1    4600 5700
-	1    0    0    1
-$EndComp
-$Comp
-L power:GND #PWR0113
-U 1 1 5E24C682
-P 4400 5900
-F 0 "#PWR0113" H 4400 5650 50  0001 C CNN
-F 1 "GND" H 4405 5727 50  0000 C CNN
-F 2 "" H 4400 5900 50  0001 C CNN
-F 3 "" H 4400 5900 50  0001 C CNN
-	1    4400 5900
-	1    0    0    -1
-$EndComp
-$Comp
-L Connector:Screw_Terminal_01x02 J5
-U 1 1 5E250E9A
-P 5050 7150
-F 0 "J5" H 5130 7142 50  0000 L CNN
-F 1 "SPINDLE_ENABLE" H 5130 7051 50  0000 L CNN
-F 2 "Connector_Phoenix_MC_HighVoltage:PhoenixContact_MC_1,5_2-G-5.08_1x02_P5.08mm_Horizontal" H 5050 7150 50  0001 C CNN
-F 3 "~" H 5050 7150 50  0001 C CNN
-	1    5050 7150
-	1    0    0    -1
-$EndComp
 Wire Wire Line
 	3550 7350 3550 7050
@@
 	5450 2800 5350 2800
 Connection ~ 5450 2550
-$Comp
-L Connector:Screw_Terminal_01x04 J6
-U 1 1 5E27D9A7
-P 6400 2050
-F 0 "J6" H 6480 2042 50  0000 L CNN
-F 1 "EMERGENCY_PROBE_ENABLE" H 6480 1951 50  0000 L CNN
-F 2 "Connector_Phoenix_MC_HighVoltage:PhoenixContact_MC_1,5_4-G-5.08_1x04_P5.08mm_Horizontal" H 6400 2050 50  0001 C CNN
-F 3 "~" H 6400 2050 50  0001 C CNN
-	1    6400 2050
-	1    0    0    -1
-$EndComp
 Wire Wire Line
 	6200 1500 6200 1950
@@
 	4400 1500 6200 1500
 Wire Wire Line
-	4400 2050 6200 2050
-Wire Wire Line
 	6100 3300 6100 2150
-Wire Wire Line
-	6100 2150 6200 2150
 Wire Wire Line
 	5350 3300 6100 3300
@@
 F 0 "J2" H 6068 5775 50  0000 C CNN
 F 1 "5V_IN" H 6068 5866 50  0000 C CNN
-F 2 "Connector_Phoenix_MC_HighVoltage:PhoenixContact_MC_1,5_2-G-5.08_1x02_P5.08mm_Horizontal" H 6150 6100 50  0001 C CNN
+F 2 "Connector_Phoenix_MC_HighVoltage:PhoenixContact_MCV_1,5_2-G-5.08_1x02_P5.08mm_Vertical" H 6150 6100 50  0001 C CNN
 F 3 "~" H 6150 6100 50  0001 C CNN
 	1    6150 6100
@@
 HV_ENABLE_B
 Wire Wire Line
-	4150 7150 4850 7150
-Wire Wire Line
-	4800 7350 4800 7250
-Wire Wire Line
-	4800 7250 4850 7250
-Wire Wire Line
 	3550 7350 4800 7350
-Text Label 4100 7350 0    50   ~ 0
+Text Label 4800 7350 0    50   ~ 0
 HV_SPINDLE_EN_B
-Text Label 4200 7150 0    50   ~ 0
+Text Label 4800 7150 0    50   ~ 0
 HV_SPINDLE_EN_A
 $Comp
@@
 	1    0    0    -1
 $EndComp
+Wire Wire Line
+	6950 1950 6200 1950
+Wire Wire Line
+	4400 2050 6950 2050
+Wire Wire Line
+	6100 2150 6950 2150
+Wire Wire Line
+	6200 2250 6950 2250
+Wire Wire Line
+	4400 5500 4850 5500
+Wire Wire Line
+	4300 5600 4850 5600
+Wire Wire Line
+	4150 5700 4850 5700
+Wire Wire Line
+	3200 5800 4850 5800
+Text Label 4850 5500 0    50   ~ 0
+PWM_A
+Text Label 4850 5600 0    50   ~ 0
+PWM_B
+Text Label 4850 5700 0    50   ~ 0
+PWM_C
+Text Label 6950 2350 2    50   ~ 0
+GND
+Text Label 6950 2450 2    50   ~ 0
+ENC
+Text Label 4850 5800 0    50   ~ 0
+ENC
+Text Label 6950 2550 2    50   ~ 0
+PWM_C
+Text Label 6950 2650 2    50   ~ 0
+PWM_B
+Text Label 6950 2750 2    50   ~ 0
+PWM_A
+Wire Wire Line
+	4800 7150 4150 7150
+Text Label 6950 2850 2    50   ~ 0
+HV_SPINDLE_EN_A
+Text Label 6950 2950 2    50   ~ 0
+HV_SPINDLE_EN_B
+Text Label 10750 3100 0    50   ~ 0
+X_DIR
+Text Label 10750 3200 0    50   ~ 0
+X_STEP
+Text Label 10750 3300 0    50   ~ 0
+Y_DIR
+Text Label 10750 3400 0    50   ~ 0
+Y_STEP
+Text Label 10750 3500 0    50   ~ 0
+Z_DIR
+Text Label 10750 3600 0    50   ~ 0
+Z_STEP
+Text Label 6950 3050 2    50   ~ 0
+Z_STEP
+Text Label 6950 3150 2    50   ~ 0
+Z_DIR
+Text Label 6950 3250 2    50   ~ 0
+Y_STEP
+Text Label 6950 3350 2    50   ~ 0
+Y_DIR
+Text Label 6950 3450 2    50   ~ 0
+X_STEP
+Text Label 6950 3550 2    50   ~ 0
+X_DIR
+$Comp
+L Connector:Screw_Terminal_01x06 J5
+U 1 1 5E7F05F7
+P 7150 2150
+F 0 "J5" H 7230 2142 50  0000 L CNN
+F 1 "Screw_Terminal_01x06" H 7230 2051 50  0000 L CNN
+F 2 "Connector_Phoenix_MC_HighVoltage:PhoenixContact_MCV_1,5_6-G-5.08_1x06_P5.08mm_Vertical" H 7150 2150 50  0001 C CNN
+F 3 "~" H 7150 2150 50  0001 C CNN
+	1    7150 2150
+	1    0    0    -1
+$EndComp
+$Comp
+L Connector:Screw_Terminal_01x11 J4
+U 1 1 5E7F24DD
+P 7150 3050
+F 0 "J4" H 7230 3092 50  0000 L CNN
+F 1 "Screw_Terminal_01x11" H 7230 3001 50  0000 L CNN
+F 2 "Connector_Phoenix_MC_HighVoltage:PhoenixContact_MCV_1,5_11-G-5.08_1x11_P5.08mm_Vertical" H 7150 3050 50  0001 C CNN
+F 3 "~" H 7150 3050 50  0001 C CNN
+	1    7150 3050
+	1    0    0    -1
+$EndComp

Commit message: vkkt
Other:
- moved on the sheet: J3
Changed lines of the file:
@@
 L Connector:DB25_Male_MountingHoles J3
 U 1 1 5E18E720
-P 1500 2600
-F 0 "J3" H 1680 2509 50  0000 L CNN
-F 1 "DB25_Male_MountingHoles" H 1680 2600 50  0000 L CNN
-F 2 "Connector_Dsub:DSUB-25_Male_Horizontal_P2.77x2.84mm_EdgePinOffset7.70mm_Housed_MountingHolesOffset9.12mm" H 1500 2600 50  0001 C CNN
-F 3 " ~" H 1500 2600 50  0001 C CNN
-	1    1500 2600
+P 1900 2150
+F 0 "J3" H 2080 2059 50  0000 L CNN
+F 1 "DB25_Male_MountingHoles" H 2080 2150 50  0000 L CNN
+F 2 "Connector_Dsub:DSUB-25_Male_Horizontal_P2.77x2.84mm_EdgePinOffset7.70mm_Housed_MountingHolesOffset9.12mm" H 1900 2150 50  0001 C CNN
+F 3 " ~" H 1900 2150 50  0001 C CNN
+	1    1900 2150
 	1    0    0    1
 $EndComp
@@
 Text Label 6350 6100 0    50   ~ 0
 LPT_VCC
-Text Label 1200 3700 2    50   ~ 0
-LPT_GND
-Text Label 1200 3500 2    50   ~ 0
-LPT_GND
-Text Label 1200 3300 2    50   ~ 0
-LPT_GND
-Text Label 1200 3100 2    50   ~ 0
-LPT_GND
-Text Label 1200 2900 2    50   ~ 0
-LPT_GND
-Text Label 1200 2700 2    50   ~ 0
-LPT_GND
-Text Label 1200 2500 2    50   ~ 0
-LPT_GND
-Text Label 1200 2300 2    50   ~ 0
-LPT_GND
-Text Label 1200 1600 2    50   ~ 0
+Text Label 1600 3250 2    50   ~ 0
+LPT_GND
+Text Label 1600 3050 2    50   ~ 0
+LPT_GND
+Text Label 1600 2850 2    50   ~ 0
+LPT_GND
+Text Label 1600 2650 2    50   ~ 0
+LPT_GND
+Text Label 1600 2450 2    50   ~ 0
+LPT_GND
+Text Label 1600 2250 2    50   ~ 0
+LPT_GND
+Text Label 1600 2050 2    50   ~ 0
+LPT_GND
+Text Label 1600 1850 2    50   ~ 0
+LPT_GND
+Text Label 1600 1150 2    50   ~ 0
 AXIS_X_DIR
-Text Label 1200 1800 2    50   ~ 0
+Text Label 1600 1350 2    50   ~ 0
 AXIS_X_STEP
-Text Label 1200 2000 2    50   ~ 0
+Text Label 1600 1550 2    50   ~ 0
 AXIS_Y_DIR
-Text Label 1200 2200 2    50   ~ 0
+Text Label 1600 1750 2    50   ~ 0
 AXIS_Y_STEP
-Text Label 1200 2400 2    50   ~ 0
+Text Label 1600 1950 2    50   ~ 0
 AXIS_Z_DIR
-Text Label 1200 2600 2    50   ~ 0
+Text Label 1600 2150 2    50   ~ 0
 AXIS_Z_STEP
-Text Label 1200 1400 2    50   ~ 0
+Text Label 1600 950  2    50   ~ 0
 ENABLE
-Text Label 1200 3600 2    50   ~ 0
+Text Label 1600 3150 2    50   ~ 0
 PROBE
-Text Label 1200 3800 2    50   ~ 0
+Text Label 1600 3350 2    50   ~ 0
 EMERGENCY
-Text Label 1200 3200 2    50   ~ 0
+Text Label 1600 2750 2    50   ~ 0
 SPINDLE_ENC
-Text Label 1200 2800 2    50   ~ 0
+Text Label 1600 2350 2    50   ~ 0
 SPINDLE_PWM
-Text Label 1200 3000 2    50   ~ 0
+Text Label 1600 2550 2    50   ~ 0
 SPINDLE_ENABLE
 $Comp
